File: EMG_Project.kicad_sch (KiCad schematic)
At the start: 73 parts, among them J1 Conn_01x03, J10 Conn_01x01, J11 Conn_01x01, J12 Conn_01x01, J13 Conn_01x01, J14 Conn_01x01, J15 Conn_01x01, J16 Conn_01x01, J18 Conn_01x01, J2 AudioJack3, J3 Conn_01x06, J4 Conn_01x01, J5 Conn_01x01, J6 Conn_01x01, J7 Conn_01x01, J8 Conn_01x01, J9 Conn_01x01, SW1 SW_SPST, U1 CJ432, U2 AMPLIFIER-INA331DGK_MSOP8, U3 OPA333AIDBVR, U4 OPA333AIDBVR, U5 ATTINY13-20SSU, U6 MP2322GQH-Z

Commit message: Assigned Footprints
Parts:
- removed J15, J16: Conn_01x01, symbol Connector_Generic:Conn_01x01
- removed J2: AudioJack3, symbol Connector_Audio:AudioJack3
- added C4: 22p, Capacitor_SMD:C_0603_1608Metric_Pad1.08x0.95mm_HandSolder, symbol Device:C
- added H1, H2, H3, H4: MountingHole, MountingHole:MountingHole_3.2mm_M3_Pad, symbol Mechanical:MountingHole
- added J12: Conn_01x02, Connector_PinHeader_2.54mm:PinHeader_1x02_P2.54mm_Horizontal, symbol Connector_Generic:Conn_01x02
- added J17: Conn_01x03, Connector_PinHeader_2.54mm:PinHeader_1x03_P2.54mm_Horizontal, symbol Connector_Generic:Conn_01x03
- added J9: SJ1-3523N, EMG Projct Footprints:CUI_SJ1-3523N, symbol SJ1-3523N:SJ1-3523N
- C1: renamed from C18; footprint (none) -> Capacitor_SMD:C_0603_1608Metric_Pad1.08x0.95mm_HandSolder
- C10: renamed from C7; footprint (none) -> Capacitor_SMD:C_0603_1608Metric_Pad1.08x0.95mm_HandSolder
- C11: renamed from C8; footprint (none) -> Capacitor_SMD:C_0603_1608Metric_Pad1.08x0.95mm_HandSolder
- C12: renamed from C11; footprint (none) -> Capacitor_SMD:C_0603_1608Metric_Pad1.08x0.95mm_HandSolder
- C13: renamed from C4; footprint (none) -> Capacitor_SMD:C_0603_1608Metric_Pad1.08x0.95mm_HandSolder
- C14: renamed from C5; footprint (none) -> Capacitor_SMD:C_0603_1608Metric_Pad1.08x0.95mm_HandSolder
- C15: renamed from C6; footprint (none) -> Capacitor_SMD:C_0603_1608Metric_Pad1.08x0.95mm_HandSolder
- C16: renamed from C9; footprint (none) -> Capacitor_SMD:C_0603_1608Metric_Pad1.08x0.95mm_HandSolder
- C17: renamed from C10; footprint (none) -> Capacitor_SMD:C_0603_1608Metric_Pad1.08x0.95mm_HandSolder
- C18: renamed from C2; footprint (none) -> Capacitor_SMD:C_0603_1608Metric_Pad1.08x0.95mm_HandSolder
- C19: renamed from C12; footprint (none) -> Capacitor_SMD:C_0603_1608Metric_Pad1.08x0.95mm_HandSolder
- C2: renamed from C16; footprint (none) -> Capacitor_SMD:C_0603_1608Metric_Pad1.08x0.95mm_HandSolder
- C20: renamed from C13; footprint (none) -> Capacitor_SMD:C_0603_1608Metric_Pad1.08x0.95mm_HandSolder
- C21: renamed from C3; footprint (none) -> Capacitor_SMD:C_0603_1608Metric_Pad1.08x0.95mm_HandSolder
- C22: renamed from C14; footprint (none) -> Capacitor_SMD:C_0603_1608Metric_Pad1.08x0.95mm_HandSolder
- C3: renamed from C20; footprint (none) -> Capacitor_SMD:C_0603_1608Metric_Pad1.08x0.95mm_HandSolder
- C5: renamed from C21; footprint (none) -> Capacitor_SMD:C_0603_1608Metric_Pad1.08x0.95mm_HandSolder
- C6: renamed from C22; footprint (none) -> Capacitor_SMD:C_0603_1608Metric_Pad1.08x0.95mm_HandSolder
- C7: renamed from C15; footprint (none) -> Capacitor_SMD:C_0603_1608Metric_Pad1.08x0.95mm_HandSolder
- C8: renamed from C19; footprint (none) -> Capacitor_SMD:C_0603_1608Metric_Pad1.08x0.95mm_HandSolder
- C9: renamed from C17; footprint (none) -> Capacitor_SMD:C_0603_1608Metric_Pad1.08x0.95mm_HandSolder
- D1: renamed from D2; footprint (none) -> LED_SMD:LED_0603_1608Metric_Pad1.05x0.95mm_HandSolder
- D2: renamed from D1; footprint (none) -> LED_SMD:LED_0603_1608Metric_Pad1.05x0.95mm_HandSolder
- J1: footprint (none) -> Connector_PinHeader_2.54mm:PinHeader_1x03_P2.54mm_Vertical
- J10: renamed from J14; footprint (none) -> Connector_PinHeader_2.54mm:PinHeader_1x01_P2.54mm_Vertical
- J11: renamed from J8; footprint (none) -> Connector_PinHeader_2.54mm:PinHeader_1x01_P2.54mm_Vertical
- J13: renamed from J5; footprint (none) -> Connector_PinHeader_2.54mm:PinHeader_1x01_P2.54mm_Vertical
- J14: renamed from J6; footprint (none) -> Connector_PinHeader_2.54mm:PinHeader_1x01_P2.54mm_Vertical
- J15: renamed from J11; footprint (none) -> Connector_PinHeader_2.54mm:PinHeader_1x01_P2.54mm_Vertical
- J16: renamed from J12; footprint (none) -> Connector_PinHeader_2.54mm:PinHeader_1x01_P2.54mm_Vertical
- J2: renamed from J3; footprint (none) -> Connector_PinHeader_2.54mm:PinHeader_1x06_P2.54mm_Horizontal
- J3: renamed from J7; footprint (none) -> Connector_PinHeader_2.54mm:PinHeader_1x01_P2.54mm_Vertical
- J4: renamed from J13; footprint (none) -> Connector_PinHeader_2.54mm:PinHeader_1x01_P2.54mm_Vertical
- J5: renamed from J10; footprint (none) -> Connector_PinHeader_2.54mm:PinHeader_1x01_P2.54mm_Vertical
- J6: renamed from J9; footprint (none) -> Connector_PinHeader_2.54mm:PinHeader_1x01_P2.54mm_Vertical
- J7: renamed from J18; footprint (none) -> Connector_PinHeader_2.54mm:PinHeader_1x01_P2.54mm_Vertical
- J8: renamed from J4; footprint (none) -> Connector_PinHeader_2.54mm:PinHeader_1x01_P2.54mm_Vertical
- L1: footprint (none) -> Inductor_SMD:L_0603_1608Metric_Pad1.05x0.95mm_HandSolder
- R1: renamed from R22; footprint (none) -> Resistor_SMD:R_0603_1608Metric_Pad0.98x0.95mm_HandSolder
- R10: renamed from R8; footprint (none) -> Resistor_SMD:R_0603_1608Metric_Pad0.98x0.95mm_HandSolder
- R11: renamed from R9; footprint (none) -> Resistor_SMD:R_0603_1608Metric_Pad0.98x0.95mm_HandSolder
- R12: footprint (none) -> Resistor_SMD:R_0603_1608Metric_Pad0.98x0.95mm_HandSolder
- R13: renamed from R10; footprint (none) -> Resistor_SMD:R_0603_1608Metric_Pad0.98x0.95mm_HandSolder
- R14: renamed from R11; footprint (none) -> Resistor_SMD:R_0603_1608Metric_Pad0.98x0.95mm_HandSolder
- R15: renamed from R14; footprint (none) -> Resistor_SMD:R_0603_1608Metric_Pad0.98x0.95mm_HandSolder
- R16: renamed from R13; footprint (none) -> Resistor_SMD:R_0603_1608Metric_Pad0.98x0.95mm_HandSolder
- R17: renamed from R18; footprint (none) -> Resistor_SMD:R_0603_1608Metric_Pad0.98x0.95mm_HandSolder
- R18: renamed from R19; footprint (none) -> Resistor_SMD:R_0603_1608Metric_Pad0.98x0.95mm_HandSolder
- R19: renamed from R17; footprint (none) -> Resistor_SMD:R_0603_1608Metric_Pad0.98x0.95mm_HandSolder
- R2: renamed from R23; footprint (none) -> Resistor_SMD:R_0603_1608Metric_Pad0.98x0.95mm_HandSolder
- R20: renamed from R4; footprint (none) -> Resistor_SMD:R_0603_1608Metric_Pad0.98x0.95mm_HandSolder
- R21: renamed from R2; footprint (none) -> Resistor_SMD:R_0603_1608Metric_Pad0.98x0.95mm_HandSolder
- R22: renamed from R3; footprint (none) -> Resistor_SMD:R_0603_1608Metric_Pad0.98x0.95mm_HandSolder
- R23: renamed from R15; value 1m -> 1M; footprint (none) -> Resistor_SMD:R_0603_1608Metric_Pad0.98x0.95mm_HandSolder
- R24: renamed from R16; footprint (none) -> Resistor_SMD:R_0603_1608Metric_Pad0.98x0.95mm_HandSolder
- R25: renamed from R20; footprint (none) -> Resistor_SMD:R_0603_1608Metric_Pad0.98x0.95mm_HandSolder
- R3: renamed from R24; footprint (none) -> Resistor_SMD:R_0603_1608Metric_Pad0.98x0.95mm_HandSolder
- R4: renamed from R25; footprint (none) -> Resistor_SMD:R_0603_1608Metric_Pad0.98x0.95mm_HandSolder
- R5: renamed from R21; footprint (none) -> Resistor_SMD:R_0603_1608Metric_Pad0.98x0.95mm_HandSolder
- R6: renamed from R1; footprint (none) -> Resistor_SMD:R_0603_1608Metric_Pad0.98x0.95mm_HandSolder
- R7: renamed from R5; footprint (none) -> Resistor_SMD:R_0603_1608Metric_Pad0.98x0.95mm_HandSolder
- R8: renamed from R7; footprint (none) -> Resistor_SMD:R_0603_1608Metric_Pad0.98x0.95mm_HandSolder
- R9: renamed from R6; footprint (none) -> Resistor_SMD:R_0603_1608Metric_Pad0.98x0.95mm_HandSolder
- SW1: footprint (none) -> Button_Switch_THT:SW_PUSH_6mm
- renumbered U6 to U1, U5 to U2, U2 to U3, U3 to U4, U4 to U5, U1 to U6
Connections:
- net GND: now also J12.2 (Pin_2)
- net REG_OUT: now also C4.1
- net V_OUT_HP: no longer J10.1 (Pin_1)
- net V_OUT_SENSOR: now also J12.1 (Pin_1)
- net S: now reaches R7.2
- net S: now also J17.3 (Pin_3), J9.1
- net R: now reaches R8.1
- net R: now also J17.2 (Pin_2), J9.3
- net T: now reaches R9.1
- net T: now also J17.1 (Pin_1), J9.2
- net at R3.2, R4.1, U1.5 (FB): now also C4.2
- net V_HP_TEST: now reaches C19.2, R23.1, R24.2
- net V_HP_TEST: now also J10.1 (Pin_1)
- net INST_INST_N renamed V_IN_INST_N
- net INST_INST_P renamed V_IN_INST_P
Other:
- note added: "???"
- note added: "Analog Frontend"
- note added: "High Frequency Rejection"
- note added: "Intrumentation Amplifer and Offset Trimming"
- note added: "Microcontroller"
- note added: "Mounting"
- note added: "Power indicator LED"
- note added: "Second amplification and filtering stage"
- note removed: "High Frequency Rejeection"
- note removed: "Intrumentation Amplifer and CM feedback net"
- note removed: "Power LED"
- moved on the sheet: C1, C10, C11, C12, C13, C14, C15, C16, C17, C18, C19, C2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

Commit message: First layout sketch
Parts:
- removed J13, J16, J3: Conn_01x01, Connector_PinHeader_2.54mm:PinHeader_1x01_P2.54mm_Vertical, symbol Connector_Generic:Conn_01x01
- added J18: Conn_01x02, Connector_PinHeader_2.54mm:PinHeader_1x02_P2.54mm_Horizontal, symbol Connector_Generic:Conn_01x02
- added R26: 0, Resistor_SMD:R_0603_1608Metric_Pad0.98x0.95mm_HandSolder, symbol Device:R
- U1: footprint EMG Projct Footprints:MP2322GQHZ -> EMG Projct Footprints:QFN-8_1p5MMx2MM_MNP
Connections:
- net +5V: now also J1.1 (Pin_1), J18.2 (Pin_2); no longer J1.3 (Pin_3)
- net GND: now also J18.1 (Pin_1)
- net REG_OUT: now also J1.3 (Pin_3); no longer J1.1 (Pin_1)
- net V_OUT_SENSOR: now also R26.1; no longer U2.2 (PB3)
- new net V_IN_MCU: R26.2, U2.2 (PB3)
Changed lines of the file:
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@@
 		)
 	)
-	(label "REG_OUT"
-		(at 49.53 204.47 0)
-		(effects
-			(font
-				(size 1.27 1.27)
-			)
-			(justify left bottom)
-		)
-	)
 	(label "TEST_LED"
 		(at 91.44 158.75 180)
@@
 		)
 	)
-	(label "V_REF"
-		(at 356.87 101.6 0)
+	(label "+5V"
+		(at 49.53 204.47 0)
 		(effects
 			(font
@@
 		)
 	)
-	(label "RST"
-		(at 91.44 153.67 180)
+	(label "V_REF"
+		(at 356.87 101.6 0)
 		(effects
 			(font
 				(size 1.27 1.27)
 			)
-			(justify right bottom)
+			(justify left bottom)
 		)
 	)
-	(label "GND"
-		(at 294.64 190.5 180)
+	(label "RST"
+		(at 91.44 153.67 180)
 		(effects
 			(font
@@
 		)
 	)
+	(label "V_IN_MCU"
+		(at 92.71 177.8 0)
+		(effects
+			(font
+				(size 1.27 1.27)
+			)
+			(justify left bottom)
+		)
+	)
 	(label "V_OUT_HP"
 		(at 546.1 208.28 0)
@@
 		)
 	)
-	(label "+5V"
-		(at 49.53 199.39 0)
-		(effects
-			(font
-				(size 1.27 1.27)
-			)
-			(justify left bottom)
-		)
-	)
 	(label "GND"
 		(at 462.28 254 180)
@@
 		)
 	)
-	(label "+3.3V"
-		(at 464.82 161.29 180)
+	(label "REG_OUT"
+		(at 49.53 199.39 0)
+		(effects
+			(font
+				(size 1.27 1.27)
+			)
+			(justify left bottom)
+		)
+	)
+	(label "+5V"
+		(at 125.73 181.61 180)
 		(effects
 			(font
@@
 		)
 	)
+	(label "V_IN_MCU"
+		(at 91.44 156.21 180)
+		(effects
+			(font
+				(size 1.27 1.27)
+			)
+			(justify right bottom)
+		)
+	)
 	(label "GND"
 		(at 152.4 180.34 180)
@@
 		)
 	)
-	(label "V_OUT_SENSOR"
-		(at 91.44 156.21 180)
+	(label "MISO"
+		(at 147.32 158.75 0)
 		(effects
 			(font
 				(size 1.27 1.27)
 			)
-			(justify right bottom)
+			(justify left bottom)
 		)
 	)
-	(label "MISO"
-		(at 147.32 158.75 0)
+	(label "GND"
+		(at 125.73 179.07 180)
 		(effects
 			(font
 				(size 1.27 1.27)
 			)
-			(justify left bottom)
+			(justify right bottom)
 		)
 	)
-	(label "GND"
-		(at 464.82 142.24 180)
+	(label "V_OUT_SENSOR"
+		(at 85.09 177.8 180)
 		(effects
 			(font
@@
 	)
 	(symbol
-		(lib_id "Connector_Generic:Conn_01x01")
-		(at 469.9 142.24 0)
-		(unit 1)
-		(exclude_from_sim no)
-		(in_bom yes)
-		(on_board yes)
-		(dnp no)
-		(fields_autoplaced yes)
-		(property "Reference" "J13"
-			(at 472.44 140.9699 0)
-			(effects
-				(font
-					(size 1.27 1.27)
-				)
-				(justify left)
-			)
-		)
-		(property "Value" "Conn_01x01"
-			(at 472.44 143.5099 0)
-			(effects
-				(font
-					(size 1.27 1.27)
-				)
-				(justify left)
-			)
-		)
-		(property "Footprint" "Connector_PinHeader_2.54mm:PinHeader_1x01_P2.54mm_Vertical"
-			(at 469.9 142.24 0)
-			(effects
-				(font
-					(size 1.27 1.27)
-				)
-				(hide yes)
-			)
-		)
-		(property "Datasheet" "~"
-			(at 469.9 142.24 0)
-			(effects
-				(font
-					(size 1.27 1.27)
-				)
-				(hide yes)
-			)
-		)
-		(property "Description" "Generic connector, single row, 01x01, script generated (kicad-library-utils/schlib/autogen/connector/)"
-			(at 469.9 142.24 0)
-			(effects
-				(font
-					(size 1.27 1.27)
-				)
-				(hide yes)
-			)
-		)
-		(property "Comments" ""
-			(at 469.9 142.24 0)
-			(effects
-				(font
-					(size 1.27 1.27)
-				)
-			)
-		)
-		(pin "1"
-		)
-		(instances
-			(project "EMG_Project"
-				(path "/2ecd8873-9ec8-4cb5-ac8f-8242dc498ac3"
-					(reference "J13")
-					(unit 1)
-				)
-			)
-		)
-	)
-	(symbol
 		(lib_id "power:GND")
 		(at 43.18 170.18 0)
@@
 	)
 	(symbol
+		(lib_id "Connector_Generic:Conn_01x02")
+		(at 130.81 179.07 0)
+		(unit 1)
+		(exclude_from_sim no)
+		(in_bom yes)
+		(on_board yes)
+		(dnp no)
+		(fields_autoplaced yes)
+		(property "Reference" "J18"
+			(at 133.35 179.0699 0)
+			(effects
+				(font
+					(size 1.27 1.27)
+				)
+				(justify left)
+			)
+		)
+		(property "Value" "Conn_01x02"
+			(at 133.35 181.6099 0)
+			(effects
+				(font
+					(size 1.27 1.27)
+				)
+				(justify left)
+			)
+		)
+		(property "Footprint" "Connector_PinHeader_2.54mm:PinHeader_1x02_P2.54mm_Horizontal"
+			(at 130.81 179.07 0)
+			(effects
+				(font
+					(size 1.27 1.27)
+				)
+				(hide yes)
+			)
+		)
+		(property "Datasheet" "~"
+			(at 130.81 179.07 0)
+			(effects
+				(font
+					(size 1.27 1.27)
+				)
+				(hide yes)
+			)
+		)
+		(property "Description" "Generic connector, single row, 01x02, script generated (kicad-library-utils/schlib/autogen/connector/)"
+			(at 130.81 179.07 0)
+			(effects
+				(font
+					(size 1.27 1.27)
+				)
+				(hide yes)
+			)
+		)
+		(pin "1"
+		)
+		(pin "2"
+		)
+		(instances
+			(project "EMG_Project"
+				(path "/2ecd8873-9ec8-4cb5-ac8f-8242dc498ac3"
+					(reference "J18")
+					(unit 1)
+				)
+			)
+		)
+	)
+	(symbol
 		(lib_id "Device:R")
 		(at 518.16 120.65 0)
@@
 	)
 	(symbol
-		(lib_id "Connector_Generic:Conn_01x01")
-		(at 469.9 161.29 0)
-		(unit 1)
-		(exclude_from_sim no)
-		(in_bom yes)
-		(on_board yes)
-		(dnp no)
-		(fields_autoplaced yes)
-		(property "Reference" "J16"
-			(at 472.44 160.0199 0)
-			(effects
-				(font
-					(size 1.27 1.27)
-				)
-				(justify left)
-			)
-		)
-		(property "Value" "Conn_01x01"
-			(at 472.44 162.5599 0)
-			(effects
-				(font
-					(size 1.27 1.27)
-				)
-				(justify left)
-			)
-		)
-		(property "Footprint" "Connector_PinHeader_2.54mm:PinHeader_1x01_P2.54mm_Vertical"
-			(at 469.9 161.29 0)
-			(effects
-				(font
-					(size 1.27 1.27)
-				)
-				(hide yes)
-			)
-		)
-		(property "Datasheet" "~"
-			(at 469.9 161.29 0)
-			(effects
-				(font
-					(size 1.27 1.27)
-				)
-				(hide yes)
-			)
-		)
-		(property "Description" "Generic connector, single row, 01x01, script generated (kicad-library-utils/schlib/autogen/connector/)"
-			(at 469.9 161.29 0)
-			(effects
-				(font
-					(size 1.27 1.27)
-				)
-				(hide yes)
-			)
-		)
-		(property "Comments" ""
-			(at 469.9 161.29 0)
-			(effects
-				(font
-					(size 1.27 1.27)
-				)
-			)
-		)
-		(pin "1"
-		)
-		(instances
-			(project "EMG_Project"
-				(path "/2ecd8873-9ec8-4cb5-ac8f-8242dc498ac3"
-					(reference "J16")
-					(unit 1)
-				)
-			)
-		)
-	)
-	(symbol
 		(lib_id "power:GND")
 		(at 209.55 194.31 0)
@@
 			)
 		)
-		(property "Footprint" "EMG Projct Footprints:MP2322GQHZ"
+		(property "Footprint" "EMG Projct Footprints:QFN-8_1p5MMx2MM_MNP"
 			(at 81.28 332.41 0)
 			(effects
@@
 	)
 	(symbol
-		(lib_id "Connector_Generic:Conn_01x01")
-		(at 299.72 190.5 0)
+		(lib_id "Device:R")
+		(at 88.9 177.8 90)
 		(unit 1)
 		(exclude_from_sim no)
@@
 		(dnp no)
 		(fields_autoplaced yes)
-		(property "Reference" "J3"
-			(at 302.26 189.2299 0)
+		(property "Reference" "R26"
+			(at 88.9 171.45 90)
 			(effects
 				(font
 					(size 1.27 1.27)
 				)
-				(justify left)
 			)
 		)
-		(property "Value" "Conn_01x01"
-			(at 302.26 191.7699 0)
+		(property "Value" "0"
+			(at 88.9 173.99 90)
 			(effects
 				(font
 					(size 1.27 1.27)
 				)
-				(justify left)
 			)
 		)
-		(property "Footprint" "Connector_PinHeader_2.54mm:PinHeader_1x01_P2.54mm_Vertical"
-			(at 299.72 190.5 0)
+		(property "Footprint" "Resistor_SMD:R_0603_1608Metric_Pad0.98x0.95mm_HandSolder"
+			(at 88.9 179.578 90)
 			(effects
 				(font
@@
 		)
 		(property "Datasheet" "~"
-			(at 299.72 190.5 0)
+			(at 88.9 177.8 0)
 			(effects
 				(font
@@
 			)
 		)
-		(property "Description" "Generic connector, single row, 01x01, script generated (kicad-library-utils/schlib/autogen/connector/)"
-			(at 299.72 190.5 0)
+		(property "Description" "Resistor"
+			(at 88.9 177.8 0)
 			(effects
 				(font
@@
 			)
 		)
-		(property "Comments" ""
-			(at 299.72 190.5 0)
-			(effects
-				(font
-					(size 1.27 1.27)
-				)
-			)
-		)
 		(pin "1"
 		)
+		(pin "2"
+		)
 		(instances
 			(project "EMG_Project"
 				(path "/2ecd8873-9ec8-4cb5-ac8f-8242dc498ac3"
-					(reference "J3")
+					(reference "R26")
 					(unit 1)
 				)

Commit message: Everything prepared for routing
Other:
- note removed: "???"
Changed lines of the file:
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@@
-		)
-	)
-	(text "???\n"
-		(exclude_from_sim no)
-		(at 304.8 118.618 0)
-		(effects
-			(font
-				(size 3.81 3.81)
-				(thickness 0.762)
-				(bold yes)
-			)
 		)
 	)
