File: EMG_Project.kicad_sch (KiCad schematic)
At the start: 77 parts, among them J1 Conn_01x03, J10 Conn_01x01, J11 Conn_01x01, J12 Conn_01x02, J14 Conn_01x01, J15 Conn_01x01, J17 Conn_01x03, J18 Conn_01x02, J2 Conn_01x06, J4 Conn_01x01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

Commit message: Added BOM and minor fixes. Revision 1 complete
Parts:
- C10, C11, C12, C13, C16, C17, C19, C20: Precision (none) -> 10%
- C14, C15: Precision (none) -> 5%
- R12, R13, R14, R15, R16, R17, R19, R21, R22, R23, R25, R8, R9: Precision (none) -> 1%
